Commit message: #3 change also urdf as well

File: eeuv_sim/urdf/Blue/base.xacro (robot description, xacro)
@@ -5,5 +5,5 @@
   <xacro:property name="cog" value="0 0 0"/>
   <xacro:property name="rho" value="1028"/>
-  <xacro:property name="visual_mesh_file" value="file://$(find uw_gazebo)/urdf/meshes/Blue/brov2_heavy_body.dae"/>
+  <xacro:property name="visual_mesh_file" value="file://$(find eeuv_sim)/urdf/meshes/Blue/brov2_heavy_body.dae"/>
   <link name="base_link">
   </link>

File: eeuv_sim/urdf/LAUV/base.xacro (robot description, xacro)
@@ -2,13 +2,13 @@
 <robot name="LAUV" xmlns:xacro="http://www.ros.org/wiki/xacro">
   <!-- Loading some constants -->
- <!-- <xacro:include filename="$(find uw_gazebo)/urdf/LAUV/common.urdf.xacro"/> -->
+ <!-- <xacro:include filename="$(find eeuv_sim)/urdf/LAUV/common.urdf.xacro"/> -->
   <!-- Loading file with sensor macros -->
-  <!-- <xacro:include filename="$(find uw_gazebo)/urdf/LAUV/sensor_snippets.xacro"/> -->
+  <!-- <xacro:include filename="$(find eeuv_sim)/urdf/LAUV/sensor_snippets.xacro"/> -->
   <!-- Loading the UUV simulator ROS plugin macros -->
-  <!--<xacro:include filename="$(find uw_gazebo)/urdf/LAUV/snippets.xacro"/> -->
+  <!--<xacro:include filename="$(find eeuv_sim)/urdf/LAUV/snippets.xacro"/> -->
   <!-- Loading vehicle's specific macros -->
-  <xacro:include filename="$(find uw_gazebo)/urdf/LAUV/common.xacro"/>
-  <xacro:include filename="$(find uw_gazebo)/urdf/LAUV/snippets.xacro"/>
-  <xacro:include filename="$(find uw_gazebo)/urdf/LAUV/gazebo.xacro"/>
+  <xacro:include filename="$(find eeuv_sim)/urdf/LAUV/common.xacro"/>
+  <xacro:include filename="$(find eeuv_sim)/urdf/LAUV/snippets.xacro"/>
+  <xacro:include filename="$(find eeuv_sim)/urdf/LAUV/gazebo.xacro"/>
   <!--
     Vehicle's parameters (remember to enter the model parameters below)
@@ -26,5 +26,5 @@
     Open the meshes for the RexROV vehicle in Blender to see an example on the mesh placement.
   -->
-  <xacro:property name="visual_mesh_file" value="file://$(find uw_gazebo)/urdf/meshes/LAUV/body.dae"/>
+  <xacro:property name="visual_mesh_file" value="file://$(find eeuv_sim)/urdf/meshes/LAUV/body.dae"/>
   <!-- Collision geometry mesh, usually in STL format (it is recommended to keep
   this geometry as simple as possible to improve the performance the physics engine
@@ -61,7 +61,7 @@
     <!-- Set up hydrodynamic plugin given as input parameter -->
     <!-- Include the thruster modules -->
-    <!-- <xacro:include filename="$(find uw_gazebo)/urdf/LAUV/actuators.xacro"/> -->
+    <!-- <xacro:include filename="$(find eeuv_sim)/urdf/LAUV/actuators.xacro"/> -->
     <!-- Include the sensor modules -->
-    <!-- <xacro:include filename="$(find uw_gazebo)/urdf/LAUV/sensors.xacro"/> -->
+    <!-- <xacro:include filename="$(find eeuv_sim)/urdf/LAUV/sensors.xacro"/> -->
   <gazebo>
     <plugin name="libgazebo_ros_p3d" filename="libgazebo_ros_p3d.so">

File: eeuv_sim/urdf/LAUV/snippets.xacro (robot description, xacro)
@@ -5,5 +5,5 @@
   over propeller's frame X-axis in DAE (Collada) or STL format.
   -->
-  <xacro:property name="prop_mesh_file" value="file://$(find uw_gazebo)/urdf/meshes/LAUV/propeller.dae"/>
+  <xacro:property name="prop_mesh_file" value="file://$(find eeuv_sim)/urdf/meshes/LAUV/propeller.dae"/>
   <!--
     Thruster macro with integration of joint and link. The thrusters should
@@ -135,6 +135,6 @@
   <!-- MACRO FOR FIN/RUDDER UNITS  -->
   <!-- A separate mesh for the fin should be stored in the meshes folder -->
-  <xacro:property name="black_fin_mesh_file" value="file://$(find uw_gazebo)/urdf/meshes/LAUV/black_fin.dae"/>
-  <xacro:property name="red_fin_mesh_file" value="file://$(find uw_gazebo)/urdf/meshes/LAUV/red_fin.dae"/>
+  <xacro:property name="black_fin_mesh_file" value="file://$(find eeuv_sim)/urdf/meshes/LAUV/black_fin.dae"/>
+  <xacro:property name="red_fin_mesh_file" value="file://$(find eeuv_sim)/urdf/meshes/LAUV/red_fin.dae"/>
   <!-- Fin properties -->
   <xacro:property name="fin_area" value="0.0064"/>

File: eeuv_sim/urdf/UCAT/base.xacro.urdf (robot description, URDF)
Before this commit: robot microcat, 5 links, 4 joints
Links:
- link sonars: geometry visual mesh filename=file://$(find eeuv_sim)/urdf/meshes/UCAT/sonar.dae scale=1 1 1; visual mesh filename=file://$(find eeuv_sim)/urdf/meshes/UCAT/sonar.dae scale=1 1 1
